File: bluegiga/eagle/BLE112/Full/BLE112 Breakout Board v2.0/BLE112 Breakout Board v2.0.sch (EAGLE design)
At the start: 27 parts, among them U1 BLE112-A, U2 MCP1700

Commit message: Fix BLE112 v2.0 trial run PCB error
Parts:
- renumbered FUSE to F1
Connections:
- net 3.3V: now also U2.VOUT; no longer U2.VO
- net GND: now also S1.2; no longer S1.3
Other:
- note added: "MCP1700T3302"
- note removed: "EXT VDD"
- note removed: "PRG VDD"
- moved on the sheet: C3
Changed lines of the file:
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@@
 </layers>
 <schematic xreflabel="%F%N/%S.%C%R" xrefpart="/%S.%C%R">
+<description>&lt;p&gt;&lt;b&gt;BLE112 Breakout Board v2.0&lt;/b&gt;&lt;/p&gt;
+&lt;p&gt;Full breakout board for all BLE112 functions, with optional LEDs, programming header, USB access, etc.&lt;/p&gt;</description>
 <attributes>
 </attributes>
@@
 </classes>
 <parts>
-<part name="FRAME1" library="frames" deviceset="FRAME_A_L" device="" value="WT12 Breakout Board v1.2"/>
+<part name="FRAME1" library="frames" deviceset="FRAME_A_L" device="" value="BLE112 Breakout Board v2.0"/>
 <part name="GND1" library="supply1" deviceset="GND" device=""/>
 <part name="U1" library="sf-bluegiga" deviceset="BLE112-A-VISUAL" device="" value="BLE112-A"/>
@@
 <part name="GND6" library="supply1" deviceset="GND" device=""/>
 <part name="GND9" library="supply1" deviceset="GND" device=""/>
-<part name="U2" library="nonolith" deviceset="MCP1700" device=""/>
 <part name="C1" library="SparkFun" deviceset="CAP" device="0603-CAP" value="0.47uF"/>
 <part name="C2" library="SparkFun" deviceset="CAP" device="0603-CAP" value="2.2uF"/>
@@
 <part name="GND13" library="supply1" deviceset="GND" device=""/>
 <part name="GND14" library="supply1" deviceset="GND" device=""/>
-<part name="FUSE" library="SparkFun" deviceset="RESISTOR" device="0805-RES" value="1K"/>
+<part name="F1" library="SparkFun" deviceset="RESISTOR" device="0805-RES" value="1K"/>
 <part name="JP3" library="adafruit" deviceset="PINHD-1X1" device="" value="5V"/>
 <part name="SJ4" library="jumper" deviceset="SJ" device="" value="EXT VDD"/>
+<part name="U2" library="nonolith" deviceset="MCP1700" device=""/>
 </parts>
 <sheets>
 <sheet>
 <plain>
-<text x="124.46" y="38.608" size="1.778" layer="91">PRG VDD</text>
 <text x="205.74" y="152.908" size="1.778" layer="91">PWR LED</text>
 <text x="205.74" y="122.428" size="1.778" layer="91">USR LED</text>
@@
 <wire x1="86.36" y1="55.88" x2="5.08" y2="55.88" width="0.1524" layer="97"/>
 <wire x1="86.36" y1="55.88" x2="86.36" y2="0" width="0.1524" layer="97"/>
-<text x="55.88" y="5.588" size="1.778" layer="91">EXT VDD</text>
+<text x="215.9" y="71.12" size="1.778" layer="91">MCP1700T3302</text>
 </plain>
 <instances>
 <instance part="FRAME1" gate="G$1" x="0" y="0"/>
 <instance part="FRAME1" gate="G$2" x="172.72" y="0"/>
-<instance part="GND1" gate="1" x="236.22" y="50.8"/>
+<instance part="GND1" gate="1" x="246.38" y="50.8"/>
 <instance part="U1" gate="G$1" x="81.28" y="139.7"/>
 <instance part="GND2" gate="1" x="58.42" y="175.26" rot="R180"/>
@@
 <instance part="PROG" gate="G$1" x="129.54" y="17.78"/>
 <instance part="U$1" gate="G$1" x="193.04" y="68.58"/>
-<instance part="P+1" gate="G$1" x="236.22" y="68.58"/>
+<instance part="P+1" gate="G$1" x="246.38" y="71.12"/>
 <instance part="U$2" gate="G$1" x="22.86" y="12.7" rot="R90"/>
 <instance part="GND7" gate="1" x="48.26" y="17.78"/>
@@
 <instance part="P+4" gate="G$1" x="119.38" y="88.9" rot="R180"/>
 <instance part="S1" gate="G$1" x="213.36" y="180.34"/>
-<instance part="GND5" gate="1" x="226.06" y="182.88" rot="R90"/>
+<instance part="GND5" gate="1" x="200.66" y="177.8" rot="R270"/>
 <instance part="R4" gate="G$1" x="213.36" y="193.04"/>
 <instance part="P+5" gate="G$1" x="223.52" y="193.04" rot="R270"/>
@@
 <instance part="SJ2" gate="1" x="210.82" y="147.32"/>
 <instance part="SJ3" gate="1" x="210.82" y="116.84"/>
-<instance part="GND4" gate="1" x="218.44" y="88.9" rot="R180"/>
+<instance part="GND4" gate="1" x="233.68" y="50.8"/>
 <instance part="GND6" gate="1" x="193.04" y="50.8"/>
 <instance part="GND9" gate="1" x="205.74" y="50.8"/>
-<instance part="U2" gate="G$1" x="218.44" y="73.66" rot="R270"/>
 <instance part="C1" gate="G$1" x="193.04" y="55.88"/>
 <instance part="C2" gate="G$1" x="205.74" y="55.88"/>
-<instance part="C3" gate="G$1" x="236.22" y="55.88"/>
+<instance part="C3" gate="G$1" x="246.38" y="55.88"/>
 <instance part="R3" gate="G$1" x="63.5" y="35.56"/>
 <instance part="C4" gate="G$1" x="50.8" y="170.18" rot="R180"/>
@@
 <instance part="GND13" gate="1" x="248.92" y="147.32" rot="R90"/>
 <instance part="GND14" gate="1" x="248.92" y="116.84" rot="R90"/>
-<instance part="FUSE" gate="G$1" x="30.48" y="12.7"/>
+<instance part="F1" gate="G$1" x="30.48" y="12.7"/>
 <instance part="JP3" gate="G$1" x="78.74" y="12.7"/>
 <instance part="SJ4" gate="1" x="60.96" y="12.7"/>
+<instance part="U2" gate="G$1" x="223.52" y="63.5"/>
 </instances>
 <busses>
@@
 <label x="111.76" y="12.7" size="1.778" layer="95"/>
 <pinref part="GND8" gate="1" pin="GND"/>
-</segment>
-<segment>
-<pinref part="S1" gate="G$1" pin="3"/>
-<pinref part="GND5" gate="1" pin="GND"/>
-<wire x1="223.52" y1="182.88" x2="220.98" y2="182.88" width="0.1524" layer="91"/>
 </segment>
 <segment>
@@
 </segment>
 <segment>
+<pinref part="GND4" gate="1" pin="GND"/>
+<wire x1="233.68" y1="53.34" x2="233.68" y2="60.96" width="0.1524" layer="91"/>
+<wire x1="233.68" y1="60.96" x2="231.14" y2="60.96" width="0.1524" layer="91"/>
 <pinref part="U2" gate="G$1" pin="GND"/>
-<pinref part="GND4" gate="1" pin="GND"/>
-<wire x1="218.44" y1="86.36" x2="218.44" y2="83.82" width="0.1524" layer="91"/>
 </segment>
 <segment>
@@
 <pinref part="C4" gate="G$1" pin="2"/>
 <pinref part="GND12" gate="1" pin="GND"/>
+</segment>
+<segment>
+<pinref part="S1" gate="G$1" pin="2"/>
+<pinref part="GND5" gate="1" pin="GND"/>
+<wire x1="203.2" y1="177.8" x2="205.74" y2="177.8" width="0.1524" layer="91"/>
 </segment>
 </net>
@@
 <junction x="205.74" y="63.5"/>
 <junction x="193.04" y="63.5"/>
-<pinref part="U2" gate="G$1" pin="VIN"/>
 <pinref part="C1" gate="G$1" pin="1"/>
 <pinref part="C2" gate="G$1" pin="1"/>
-</segment>
-<segment>
-<pinref part="FUSE" gate="G$1" pin="1"/>
+<pinref part="U2" gate="G$1" pin="VIN"/>
+</segment>
+<segment>
+<pinref part="F1" gate="G$1" pin="1"/>
 <pinref part="U$2" gate="G$1" pin="5V"/>
 <wire x1="22.86" y1="12.7" x2="25.4" y2="12.7" width="0.1524" layer="91"/>
@@
 <net name="3.3V" class="1">
 <segment>
-<wire x1="220.98" y1="63.5" x2="236.22" y2="63.5" width="0.1524" layer="91"/>
-<wire x1="236.22" y1="63.5" x2="236.22" y2="60.96" width="0.1524" layer="91"/>
-<wire x1="236.22" y1="63.5" x2="236.22" y2="68.58" width="0.1524" layer="91"/>
-<junction x="236.22" y="63.5"/>
+<wire x1="231.14" y1="66.04" x2="246.38" y2="66.04" width="0.1524" layer="91"/>
+<wire x1="246.38" y1="66.04" x2="246.38" y2="60.96" width="0.1524" layer="91"/>
+<wire x1="246.38" y1="66.04" x2="246.38" y2="71.12" width="0.1524" layer="91"/>
+<junction x="246.38" y="66.04"/>
 <pinref part="P+1" gate="G$1" pin="3.3V"/>
-<pinref part="U2" gate="G$1" pin="VO"/>
 <pinref part="C3" gate="G$1" pin="1"/>
+<pinref part="U2" gate="G$1" pin="VOUT"/>
 </segment>
 <segment>
@@
 <pinref part="SJ1" gate="1" pin="2"/>
 <wire x1="149.86" y1="33.02" x2="149.86" y2="35.56" width="0.1524" layer="91"/>
-<wire x1="134.62" y1="33.02" x2="137.16" y2="33.02" width="0.1524" layer="91"/>
-<wire x1="137.16" y1="33.02" x2="149.86" y2="33.02" width="0.1524" layer="91"/>
-<wire x1="137.16" y1="38.1" x2="137.16" y2="33.02" width="0.1524" layer="91" style="shortdash"/>
-<junction x="137.16" y="33.02"/>
+<wire x1="134.62" y1="33.02" x2="149.86" y2="33.02" width="0.1524" layer="91"/>
 <junction x="149.86" y="33.02"/>
 </segment>
@@
 <wire x1="71.12" y1="22.86" x2="40.64" y2="22.86" width="0.1524" layer="91"/>
 <wire x1="40.64" y1="22.86" x2="40.64" y2="12.7" width="0.1524" layer="91"/>
-<pinref part="FUSE" gate="G$1" pin="2"/>
+<pinref part="F1" gate="G$1" pin="2"/>
 <wire x1="40.64" y1="12.7" x2="35.56" y2="12.7" width="0.1524" layer="91"/>
 <pinref part="SJ4" gate="1" pin="1"/>
-<wire x1="55.88" y1="12.7" x2="53.34" y2="12.7" width="0.1524" layer="91"/>
-<wire x1="53.34" y1="12.7" x2="40.64" y2="12.7" width="0.1524" layer="91"/>
-<wire x1="53.34" y1="12.7" x2="53.34" y2="5.08" width="0.1524" layer="91" style="shortdash"/>
-<junction x="53.34" y="12.7"/>
+<wire x1="55.88" y1="12.7" x2="40.64" y2="12.7" width="0.1524" layer="91"/>
 <junction x="40.64" y="12.7"/>
 </segment>
@@
 <wire x1="121.92" y1="22.86" x2="109.22" y2="22.86" width="0.1524" layer="91"/>
 <pinref part="SJ1" gate="1" pin="1"/>
-<wire x1="124.46" y1="33.02" x2="121.92" y2="33.02" width="0.1524" layer="91"/>
-<wire x1="121.92" y1="33.02" x2="121.92" y2="38.1" width="0.1524" layer="91" style="shortdash"/>
-<junction x="121.92" y="33.02"/>
-<wire x1="121.92" y1="33.02" x2="109.22" y2="33.02" width="0.1524" layer="91"/>
+<wire x1="124.46" y1="33.02" x2="109.22" y2="33.02" width="0.1524" layer="91"/>
 <wire x1="109.22" y1="33.02" x2="109.22" y2="22.86" width="0.1524" layer="91"/>
 <label x="111.76" y="22.86" size="1.778" layer="95"/>
@@
 <pinref part="JP3" gate="G$1" pin="1"/>
 <pinref part="SJ4" gate="1" pin="2"/>
-<wire x1="66.04" y1="12.7" x2="68.58" y2="12.7" width="0.1524" layer="91"/>
-<wire x1="68.58" y1="12.7" x2="76.2" y2="12.7" width="0.1524" layer="91"/>
-<junction x="68.58" y="12.7"/>
-<wire x1="68.58" y1="5.08" x2="68.58" y2="12.7" width="0.1524" layer="91" style="shortdash"/>
-</segment>
-</net>
+<wire x1="66.04" y1="12.7" x2="76.2" y2="12.7" width="0.1524" layer="91"/>
+</segment>
+</net>
